File: JeppRadiocomandataARDUINO/Hardware/JeepPCB/JeepPCB.kicad_sch (KiCad schematic)
At the start: 21 parts, among them J1 Radio, U1 ATmega328P-A, Y1 Crystal

Commit message: Aggiornamento delle tracce
Connections:
- net INO_D10: now also MotorFET1.5 (IN1); no longer MotorFET1.6 (EnA)
- net INO_D5: now also MotorFET1.12 (IN4); no longer MotorFET1.11 (EnB)
- net INO_D6: now also MotorFET1.11 (EnB); no longer MotorFET1.12 (IN4)
- net INO_D9: now also MotorFET1.6 (EnA); no longer MotorFET1.5 (IN1)
Changed lines of the file:
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@@
     (effects (font (size 1.27 1.27)) (justify left bottom))
   )
-  (global_label "INO_D10" (shape input) (at 65.532 39.878 180) (fields_autoplaced)
+  (global_label "INO_D10" (shape input) (at 65.532 34.798 180) (fields_autoplaced)
     (effects (font (size 0.8 0.8)) (justify right))
-    (property "Intersheet References" "${INTERSHEET_REFS}" (id 0) (at 59.0215 39.828 0)
+    (property "Intersheet References" "${INTERSHEET_REFS}" (id 0) (at 59.0215 34.748 0)
       (effects (font (size 0.8 0.8)) (justify right) hide)
     )
   )
-  (global_label "INO_D6" (shape input) (at 65.532 47.498 180) (fields_autoplaced)
+  (global_label "INO_D6" (shape input) (at 65.532 50.038 180) (fields_autoplaced)
     (effects (font (size 0.8 0.8)) (justify right))
-    (property "Intersheet References" "${INTERSHEET_REFS}" (id 0) (at 59.7834 47.448 0)
+    (property "Intersheet References" "${INTERSHEET_REFS}" (id 0) (at 59.7834 49.988 0)
       (effects (font (size 0.8 0.8)) (justify right) hide)
     )
@@
     )
   )
-  (global_label "INO_D5" (shape input) (at 65.532 50.038 180) (fields_autoplaced)
+  (global_label "INO_D5" (shape input) (at 65.532 47.498 180) (fields_autoplaced)
     (effects (font (size 0.8 0.8)) (justify right))
-    (property "Intersheet References" "${INTERSHEET_REFS}" (id 0) (at 59.7834 49.988 0)
+    (property "Intersheet References" "${INTERSHEET_REFS}" (id 0) (at 59.7834 47.448 0)
       (effects (font (size 0.8 0.8)) (justify right) hide)
     )
@@
     )
   )
-  (global_label "INO_D9" (shape input) (at 65.532 34.798 180) (fields_autoplaced)
+  (global_label "INO_D9" (shape input) (at 65.532 39.878 180) (fields_autoplaced)
     (effects (font (size 0.8 0.8)) (justify right))
-    (property "Intersheet References" "${INTERSHEET_REFS}" (id 0) (at 59.7834 34.748 0)
+    (property "Intersheet References" "${INTERSHEET_REFS}" (id 0) (at 59.7834 39.828 0)
       (effects (font (size 0.8 0.8)) (justify right) hide)
     )

Commit message: Jeep Finita
Parts:
- renumbered REG_LIN1 to RL1
Changed lines of the file:
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@@
   (symbol (lib_id "Regulator_Linear:KA78M05_TO252") (at 48.006 49.022 0) (unit 1)
     (in_bom yes) (on_board yes)
-    (property "Reference" "REG_LIN1" (id 0) (at 47.752 45.466 0))
+    (property "Reference" "RL1" (id 0) (at 47.752 45.466 0))
     (property "Value" "KA78M05_TO252" (id 1) (at 48.006 44.196 0)
       (effects (font (size 1.27 1.27)) hide)
@@
     )
     (path "/eb166358-be61-4056-b159-d0aba37bef05"
-      (reference "REG_LIN1") (unit 1) (value "KA78M05_TO252") (footprint "Package_TO_SOT_SMD:TO-252-2")
+      (reference "RL1") (unit 1) (value "KA78M05_TO252") (footprint "Package_TO_SOT_SMD:TO-252-2")
     )
     (path "/c751029c-0ca6-4cd0-8725-946b9af36995"
