File: JeppRadiocomandataARDUINO/Hardware/JeepPCB/JeepPCB.kicad_sch (KiCad schematic)
At the start: 21 parts, among them J1 Radio, U1 ATmega328P-A, Y1 Crystal

Commit message: Aggiornamento del PCB aggiunta di VCC e di Vie
Parts:
- C1, C2: footprint Capacitor_SMD:C_Elec_4x5.8 -> Capacitor_SMD:C_Elec_8x10.2
- J1: footprint Connector_PinHeader_1.00mm:PinHeader_1x03_P1.00mm_Vertical -> Connector_PinHeader_2.00mm:PinHeader_1x03_P2.00mm_Vertical
Changed lines of the file:
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@@
       (effects (font (size 1.27 1.27)) (justify left))
     )
-    (property "Footprint" "Capacitor_SMD:C_Elec_4x5.8" (id 2) (at 24.638 57.658 0)
+    (property "Footprint" "Capacitor_SMD:C_Elec_8x10.2" (id 2) (at 24.638 57.658 0)
       (effects (font (size 1.27 1.27)) hide)
     )
@@
       (effects (font (size 1.27 1.27)) (justify right))
     )
-    (property "Footprint" "Connector_PinHeader_1.00mm:PinHeader_1x03_P1.00mm_Vertical" (id 2) (at 154.178 145.288 0)
+    (property "Footprint" "Connector_PinHeader_2.00mm:PinHeader_1x03_P2.00mm_Vertical" (id 2) (at 154.178 145.288 0)
       (effects (font (size 1.27 1.27)) hide)
     )
@@
       (effects (font (size 1.27 1.27)) (justify left))
     )
-    (property "Footprint" "Capacitor_SMD:C_Elec_4x5.8" (id 2) (at 55.626 57.658 0)
+    (property "Footprint" "Capacitor_SMD:C_Elec_8x10.2" (id 2) (at 55.626 57.658 0)
       (effects (font (size 1.27 1.27)) hide)
     )
@@
     )
     (path "/d009009f-95c2-4e0c-9edf-2151737e2628"
-      (reference "C1") (unit 1) (value "220uF") (footprint "Capacitor_SMD:C_Elec_4x5.8")
+      (reference "C1") (unit 1) (value "220uF") (footprint "Capacitor_SMD:C_Elec_8x10.2")
     )
     (path "/042c4ba9-5cce-4d89-8fe4-3f031769c4bf"
-      (reference "C2") (unit 1) (value "220uF") (footprint "Capacitor_SMD:C_Elec_4x5.8")
+      (reference "C2") (unit 1) (value "220uF") (footprint "Capacitor_SMD:C_Elec_8x10.2")
     )
     (path "/81c0867b-d819-4bc6-8926-eccf1eda061e"
@@
     )
     (path "/c6ff950c-fe73-4725-a0da-2103c5405644"
-      (reference "J1") (unit 1) (value "Radio") (footprint "Connector_PinHeader_1.00mm:PinHeader_1x03_P1.00mm_Vertical")
+      (reference "J1") (unit 1) (value "Radio") (footprint "Connector_PinHeader_2.00mm:PinHeader_1x03_P2.00mm_Vertical")
     )
     (path "/09740267-1ffb-4c95-a882-d84ec24f41f1"

Commit message: Foot Print del processore a 8 bit che verrà utilizzato al posto di ATMega328P
Other:
- company: (none) -> Giovanni Rasera
Changed lines of the file:
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@@
   (title_block
     (title "Jepp Radiocomandata")
-    (date "2022-06-21")
+    (date "2022-06-29")
     (rev "1.0.0")
-    (comment 1 "Giovanni Rasera")
+    (company "Giovanni Rasera")
   )
   (junction (at 131.826 19.304) (diameter 0) (color 0 0 0 0)
