File: DronePCB/DroneHardware/Power.kicad_sch (KiCad schematic)
At the start: 17 parts, among them Q101 AO3401A, U101 MP2359DJ-LF-Z

Commit message: Posizionamento di tutte le componenti
Changed lines of the file:
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@@
   (symbol (lib_id "Device:D_Schottky_Small") (at 45.466 78.486 90) (unit 1)
     (in_bom yes) (on_board yes)
-    (property "Reference" "D101" (id 0) (at 50.038 78.486 90)
+    (property "Reference" "D101" (id 0) (at 46.736 84.582 90)
       (effects (font (size 1.27 1.27)) (justify left))
     )
