File: DronePCB/DroneHardware/DroneHardware.kicad_pcb (KiCad board)
At the start: 6 copper layers, 36.1 x 36 mm, 49 parts, among them J201 USB_B_Micro, J202 BATTERY, J203 SWD_CONN, Q101 AO3401A, SW1 SW_SPDT, U1 STM32F405RGT6, U101 MP2359DJ-LF-Z, U201 USBLC6-2SC6, U301 MPU-6000, Y1 16MHz

Commit message: Aggiornamento delle tracce
Parts:
- moved C3 16.9 mm to (176.8, 47.1)
Routing:
- net +5V: track 6.43 -> 53.5 mm, vias 0 -> 2
- net USB_D-: track 0.00 -> 28.5 mm, vias 0 -> 2
- net SWCLK: track 0.00 -> 25.7 mm, vias 0 -> 2
- net SWO: track 0.00 -> 24.3 mm
- net SWDIO: track 0.00 -> 23.9 mm, vias 0 -> 2
- net NRST: track 0.00 -> 22.8 mm
- net USB_D+: track 0.00 -> 22.1 mm, vias 0 -> 2
- net unconnected-(J201-Pad6): track 0.00 -> 11.5 mm
- net GND: track 44.5 -> 52.5 mm, vias 29 -> 35
- net BUCK_VOUT_3V3: track 26.0 -> 31.6 mm, vias 7 -> 13
- net HSE_OUT: track 2.85 -> 3.50 mm
