File: DronePCB/5V_DroneHardware/Gyro.kicad_sch (KiCad schematic)
At the start: 4 parts, among them U303 MPU-6000

Commit message: BOM e pos file
Parts:
- C317: LCSC Part # C15195 -> C1532
- U303: LCSC Part # (none) -> C92401
Changed lines of the file:
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@@
+      (effects (font (size 1.27 1.27)) hide)
+    )
+    (property "LCSC Part #" "C92401" (id 4) (at 146.304 100.838 0)
       (effects (font (size 1.27 1.27)) hide)
     )
@@
       (effects (font (size 1.27 1.27)) hide)
     )
-    (property "LCSC Part #" "C15195" (id 4) (at 178.054 110.998 0)
+    (property "LCSC Part #" "C1532" (id 4) (at 178.054 110.998 0)
       (effects (font (size 1.27 1.27)) hide)
     )
